File: tag_connect_adaptor.kicad_pcb (KiCad board)
At the start: 2 copper layers, 108 x 93.5 mm, 10 parts, among them J1 INPUT, J2 OUTPUT, J3 ISP-USBASP, J4 ST-LINK CLONE, J5 TAG 6 PIN, SW1 BYPASS

Commit message: Numpering update
Other:
- board text added: "JLCJLCJLCJLC"
Changed lines of the file:
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@@
   (general
     (thickness 1.6)
-    (drawings 13)
+    (drawings 14)
     (tracks 104)
     (zones 0)
@@
     )
   )
+  (gr_text JLCJLCJLCJLC (at 22 68) (layer F.SilkS)
+    (effects (font (size 1 1) (thickness 0.15)))
+  )
   (gr_text "Yiancar-Designs\nTag Connect Patch Module" (at 101 108) (layer F.SilkS)
